File: fpga_linux.sch (EAGLE design)
At the start: 85 parts, among them IC1 E1109AFGB, IC2 LFE5U-25F68G256CFDG

Commit message: Added gregs recommendations (pullup/down on grogramn/tck, usrled)
Parts:
- added LED1: (no value), led:LEDCHIP-LED0603
- added R31, R32, R33: (no value), my_lib:R0402
Connections:
- removed net RAM_DU: IC2G$5.PR8C
- new net LED_N: IC2G$8.PL8B, LED1.C
- new net N$2: LED1.A, R33.1
- net +3V3: now also R31.1, R33.2
- net GND: now also R32.2
- net RAM_A13: now also IC2G$6.PR38C; no longer IC2G$6.PR35B/VREF1_3
- net RAM_D3: now also IC2G$5.PR8C; no longer IC2G$5.PR11A
- net RAM_RAS_N: now also IC2G$5.PR5D; no longer IC2G$5.PR14C/VREF1_2
- net RESET_N: now also R31.2
- net TCK: now also R32.1
- net VTT: now also IC2G$5.PR14C/VREF1_2, IC2G$6.PR35B/VREF1_3
Other:
- moved on the sheet: IC2G$2, JP2
